File: e77/e77.kicad_sch (KiCad schematic)
At the start: 18 parts, among them J1 Conn_01x06_Pin, J2 Conn_01x06_Pin, U1 XBEE_MODULE, U2 XBEE_MODULE, U3 E77, U4 Rak3172

Commit message: add Radiohead_Lib
Parts:
- RN2: value 10k -> 4k7
Changed lines of the file:
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@@
 			)
 		)
-		(property "Value" "10k"
+		(property "Value" "4k7"
 			(at 168.91 138.43 90)
 			(effects
